File: EDA/EDA/microBoSL.sch (KiCad schematic (older format))
At the start: 67 parts, among them CON1 Micro_SD_Card, CON2 BARREL_JACK, IC2 SIM7000, J1 Screw_Terminal_1x06, J10 Conn_01x08, J2 Screw_Terminal_1x04, J3 Screw_Terminal_1x02, J4 Screw_Terminal_1x08, J5 Screw_Terminal_1x04, J6 RJ45, J7 USB_B_Micro, J8 Conn_01x05, J9 Conn_01x06, P2 CONN_01X04, P3 CONN_01X04, P4 CONN_01X04, SW1 SPST, U1 MCP1700T-3302E/TT, U2 MS5803, U3 MSQA6V1W5T2G, U4 74HC126, U5 FT232RL, U6 ATmega328P-AU, U7 MCP7940N-xSN, Y1 8 MHz, Y2 32.768 kHz

Commit message: chnaged a few packages arround
Parts:
- removed J1: Screw_Terminal_1x06, TerminalBlock_Phoenix:TerminalBlock_Phoenix_PT-1,5-6-3.5-H_1x06_P3.50mm_Horizontal, symbol SIM7000-rescue:Screw_Terminal_1x06-SIM7000-rescue
- removed J10: Conn_01x08, Connector_PinHeader_2.54mm:PinHeader_1x08_P2.54mm_Vertical, symbol Connector_Generic:Conn_01x08
- removed J2, J5: Screw_Terminal_1x04, TerminalBlock_Phoenix:TerminalBlock_Phoenix_PT-1,5-4-3.5-H_1x04_P3.50mm_Horizontal, symbol SIM7000-rescue:Screw_Terminal_1x04-SIM7000-rescue
- removed J3: Screw_Terminal_1x02, TerminalBlock_Phoenix:TerminalBlock_Phoenix_PT-1,5-2-3.5-H_1x02_P3.50mm_Horizontal, symbol SIM7000-rescue:Screw_Terminal_1x02-SIM7000-rescue
- removed J4: Screw_Terminal_1x08, TerminalBlock_Phoenix:TerminalBlock_Phoenix_PT-1,5-8-3.5-H_1x08_P3.50mm_Horizontal, symbol SIM7000-rescue:Screw_Terminal_1x08-SIM7000-rescue
- removed J6: RJ45, SIMFootprints:RJ_45, symbol SIM7000-rescue:RJ45-SIM7000-rescue
- removed J8: Conn_01x05, Connector_PinHeader_2.54mm:PinHeader_1x05_P2.54mm_Vertical, symbol Connector_Generic:Conn_01x05
- removed J9: Conn_01x06, Connector_PinHeader_2.54mm:PinHeader_1x06_P2.54mm_Vertical, symbol Connector_Generic:Conn_01x06
- removed P2, P3, P4: CONN_01X04, Connector_PinHeader_2.54mm:PinHeader_1x04_P2.54mm_Vertical, symbol SIM7000-rescue:CONN_01X04-SIM7000-rescue
- C10, C11, C12, C2, C3, C4, C8, C9: footprint Capacitor_SMD:C_0805_2012Metric -> Capacitor_SMD:C_0603_1608Metric
- D2, D3, D4, D5, D6: footprint LED_SMD:LED_0805_2012Metric -> LED_SMD:LED_0603_1608Metric
- R1, R2, R3, R4, R5, R6, R7, R8, R9: footprint Resistor_SMD:R_0805_2012Metric -> Resistor_SMD:R_0603_1608Metric
- U6: footprint Package_QFP:TQFP-32_7x7mm_P0.8mm -> Package_DFN_QFN:QFN-32-1EP_5x5mm_P0.5mm_EP3.1x3.1mm
Other:
- note added: "RFID"
- note removed: "Eithernet Sensor Port"
- note removed: "Peripheral Connectivity"

Commit message: added new footprints
Parts:
- removed IC2: SIM7000, SIMFootprints:SIM7000, symbol SIM7000-rescue:SIM7000-simcom
- removed R2, R3: 10 kΩ, Resistor_SMD:R_0603_1608Metric, symbol Device:R
- removed TP2, TP3: TEST, TestPoint:TestPoint_Pad_D1.0mm, symbol SIM7000-rescue:TEST-SIM7000-rescue
- removed TP4, TP5, TP6, TP7: TestPoint, TestPoint:TestPoint_Pad_1.5x1.5mm, symbol Connector:TestPoint
- removed U2: MS5803, SIMFootprints:MS5803, symbol SIM7000-rescue:MS5803-simcom
- removed U5: FT232RL, Package_SO:SSOP-28_5.3x10.2mm_P0.65mm, symbol SIM7000-rescue:FT232RL-simcom
- added TP? (x5): TEST, TestPoint:TestPoint_Pad_D1.0mm, symbol SIM7000-rescue:TEST-SIM7000-rescue
- added U5: FT232RQ, Package_DFN_QFN:QFN-32-1EP_5x5mm_P0.5mm_EP3.1x3.1mm, symbol SIM7000-rescue:FT232RQ
- added U?: SIM7090, symbol SIM7000-rescue:SIM7090
- added U? (x2): 74LV1T34GXH, symbol SIM7000-rescue:74LV1T34GXH
- U4: footprint Package_SO:SOIC-14_3.9x8.7mm_P1.27mm -> Package_SO:TSSOP-14_4.4x5mm_P0.65mm
- U7: footprint Package_SO:SOIC-8_3.9x4.9mm_P1.27mm -> Package_DFN_QFN:DFN-8-1EP_3x2mm_P0.5mm_EP1.3x1.5mm
Connections:
- net AND_RX: now also U5.30 (TXD)
- net AND_TX: now also U5.2 (RXD)
- net GND: now also C8.1, U5.17 (GND), U5.20 (GND), U5.24 (AGND), U5.4 (GND), U?.22 (GND), U?.23 (GND), U?.24 (GND), U?.25 (GND), U?.27 (GND), U?.28 (GND), U?.3 (GND), U?.3 (GND), U?.30 (GND), U?.31 (GND), U?.43 (GND), U?.47 (GND), U?.52 (GND), U?.53 (GND), U?.54 (GND), U?.55 (GND), U?.56 (GND), U?.58 (GND), U?.65 (GND), U?.66 (GND), U?.73 (GND), U?.74 (GND), U?.75 (GND), U?.84 (GND), U?.85 (GND), U?.86 (GND), U?.88 (GND), U?.89 (GND); no longer C8.2
- net NETLIGHT: now also U?.79 (NETLIGHT)
- net PWR_STAT: now also U?.78 (STATUS)
- net RX: now also U?.4 (Y)
- net TTL_3.3V: now also C8.2, U5.1 (VCCIO), U5.16 (3V3OUT); no longer C8.1
- net TX: now also U?.2 (A)
- net USB_DM: now also U5.15 (USBD-)
- net USB_DP: now also U5.14 (USBD+)
- net USB_V: now also U5.19 (VCC)
- net VPP: now also U?.19 (VBAT), U?.20 (VBAT)
- net V_3.3: now also U?.5 (VCC)
- net at D1.2 (A), TP1.1: now also U?.46 (PWRKEY)
- net at C4.2, I1.1 (VCC), U3.5: now also U?.16 (USIM_VDD)
- net at U3.4: now also I1.2 (RST), U?.15 (USIM_RST); no longer I1.6 (DATA)
- net at I1.3 (CLK): now also U3.1, U?.13 (USIM_CLK); no longer U3.3
- net at C10.2: now also U?.32 (ANT_GNSS)
- net at AT3.1: now also U?.26 (ANT_MAIN)
- net at C9.2: now also U5.31 (DTR)
- net at R8.2: now also U5.21 (CBUS1)
- net at R7.2: now also U5.22 (CBUS0)
- new net: I1.6 (DATA), U3.3, U?.14 (USIM_DATA)
- new net: TP?.1, U?.10 (USB_DM)
- new net: TP?.1, U?.11 (USB_DP)
- new net: TP?.1, U?.12 (USB_VBUS)
- new net: U?.4 (Y), U?.6 (RXD)
- new net: U?.2 (A), U?.7 (TXD)
- new net: TP?.1, U?.87 (BOOT_CFG)
- new net V_1.8: TP?.1, U?.21 (VDD_EXT), U?.5 (VCC)
- no-connect marks 38 -> 15
Other:
- note added: "50 Ω"
- note removed: "SIM 7000 USB Debug"
- moved on the sheet: AT2, AT3, C10, C4, C5, C6, C7, C8, C9, D1, D4, D5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
