File: nano/EDA/EDA/BoSLnano.sch (KiCad schematic (older format))
At the start: 59 parts, among them J1 Micro_SD_Card, J2 Conn_02x04_Counter_Clockwise, J3 Barrel_Jack_Switch, J4 USB_B_Micro, SW1 SPST, U1 MCP1700-3302E_SOT23, U10 FT232RQ, U2 ATmega328P-MMH, U3 MSQA6V1W5T2G, U4 NT3H2111W0FTT, U5 SIM7090, U6 74LV1T34GXH, U7 74LV1T34GXH, U8 MCP7940N-xSN, U9 74HC126PW-Q100, Y1 8 MHz, Y2 32.768 kHz

Commit message: finished bom and schematic - nano
Parts:
- removed BT1: Battery_Cell, SIMFootprints:2996TR, symbol Device:Battery_Cell
- removed C1: 0.1 μF, Capacitor_SMD:C_0805_2012Metric, symbol Device:C
- removed C10, C9: 12 pF, Capacitor_SMD:C_0603_1608Metric, symbol Device:C
- removed C11, C12: 100 nF, Capacitor_SMD:C_0603_1608Metric, symbol Device:C
- removed C2: 1 μF, Capacitor_SMD:C_1206_3216Metric, symbol Device:C
- removed C5, C6: 22 pF, Capacitor_SMD:C_0603_1608Metric, symbol Device:C
- removed C8: 33 pF, Capacitor_SMD:C_0603_1608Metric, symbol Device:C
- removed D1: 1N4148, Diode_SMD:D_SOD-323, symbol Device:D
- removed D4, D5: LED, LED_SMD:LED_0603_1608Metric, symbol Device:LED
- removed J2: Conn_02x04_Counter_Clockwise, Connector_PinHeader_2.54mm:PinHeader_2x04_P2.54mm_Vertical, symbol Connector_Generic:Conn_02x04_Counter_Clockwise
- removed R7: 10 kΩ, Resistor_SMD:R_0603_1608Metric, symbol Device:R
- removed R8, R9: 3.3 kΩ, Resistor_SMD:R_0603_1608Metric, symbol Device:R
- removed TP1: PWR_KEY, TestPoint:TestPoint_Pad_D1.0mm, symbol SIM7000-rescue:TEST-SIM7000-rescue
- removed TP2: VDD_EXT, TestPoint:TestPoint_Pad_D1.0mm, symbol SIM7000-rescue:TEST-SIM7000-rescue
- removed TP3: USB_DM, TestPoint:TestPoint_Pad_D1.0mm, symbol SIM7000-rescue:TEST-SIM7000-rescue
- removed TP4: USB_DP, TestPoint:TestPoint_Pad_D1.0mm, symbol SIM7000-rescue:TEST-SIM7000-rescue
- removed TP5: USB_VBUS, TestPoint:TestPoint_Pad_D1.0mm, symbol SIM7000-rescue:TEST-SIM7000-rescue
- removed TP6: BOOT_CFG, TestPoint:TestPoint_Pad_D1.0mm, symbol SIM7000-rescue:TEST-SIM7000-rescue
- removed U10: FT232RQ, Package_DFN_QFN:QFN-32-1EP_5x5mm_P0.5mm_EP3.1x3.1mm, symbol SIM7000-rescue:FT232RQ
- removed U2: ATmega328P-MMH, Package_DFN_QFN:QFN-28-1EP_4x4mm_P0.45mm_EP2.4x2.4mm, symbol MCU_Microchip_ATmega:ATmega328P-MMH
- removed U5: SIM7090, SIMFootprints:SIM9000, symbol SIM7000-rescue:SIM7090
- removed U6, U7: 74LV1T34GXH, SIMFootprints:SOT1226, symbol SIM7000-rescue:74LV1T34GXH
- removed U8: MCP7940N-xSN, Package_DFN_QFN:DFN-8-1EP_3x2mm_P0.5mm_EP1.3x1.5mm, symbol Timer:MCP7940N-xSN
- removed U9: 74HC126PW-Q100, Package_SO:TSSOP-14_4.4x5mm_P0.65mm, symbol SIM7000-rescue:74HC126
- removed Y1: 8 MHz, Crystal:Crystal_SMD_EuroQuartz_MT-4Pin_3.2x2.5mm, symbol Device:Crystal
- removed Y2: 32.768 kHz, Crystal:Crystal_SMD_EuroQuartz_EQ161-2Pin_3.2x1.5mm, symbol Device:Crystal
- added C10, C11, C12, C15, C18, C3, C6, C7, C8: 100 nF, Capacitor_SMD:C_0402_1005Metric, symbol Device:C_Small
- added C13, C16, C4, C5: 15 pF, Capacitor_SMD:C_0402_1005Metric, symbol Device:C_Small
- added C14, C9: 1 μF, Capacitor_SMD:C_0402_1005Metric, symbol Device:C_Small
- added C19: 1 nF, Capacitor_SMD:C_0402_1005Metric, symbol Device:C_Small
- added D1: D_Schottky, SIMFootprints:SOD882, symbol Device:D_Schottky
- added J2: Conn_01x07, Connector_PinHeader_2.54mm:PinHeader_1x07_P2.54mm_Vertical, symbol Connector_Generic:Conn_01x07
- added J3, J7: Conn_01x04, Connector_PinHeader_2.54mm:PinHeader_1x04_P2.54mm_Vertical, symbol Connector_Generic:Conn_01x04
- added J4: SAMD_DBG, SIMFootprints:TC2030, symbol Connector_Generic:Conn_02x03_Odd_Even
- added J5: nRF_DBG, SIMFootprints:TC2030, symbol Connector_Generic:Conn_02x03_Odd_Even
- added J6: Conn_01x10, Connector_PinHeader_2.54mm:PinHeader_1x10_P2.54mm_Vertical, symbol Connector_Generic:Conn_01x10
- added L1: 9.1 nH, Inductor_SMD:L_0603_1608Metric, symbol Device:L
- added R1, R2: 1 kΩ, Resistor_SMD:R_0402_1005Metric, symbol Device:R
- added R12, R13, R14, R15: 10 kΩ, Resistor_SMD:R_0402_1005Metric, symbol Device:R
- added R3: 39 Ω, Resistor_SMD:R_0402_1005Metric, symbol Device:R
- added R4: 100 kΩ, Resistor_SMD:R_0402_1005Metric, symbol Device:R
- added U2: ATSAMD21G18A-MUT, Package_DFN_QFN:QFN-48-1EP_7x7mm_P0.5mm_EP5.15x5.15mm, symbol MCU_Microchip_SAMD:ATSAMD21G18A-AUT
- added U4: NRF9160, symbol SIM7000-rescue:NRF9160
- added U5: BGA524N6, SIMFootprints:TSNP-6-2, symbol SIM7000-rescue:BGA524N6
- added Y1: 32.768kHz, Crystal:Crystal_SMD_EuroQuartz_EQ161-2Pin_3.2x1.5mm, symbol Device:Crystal_Small
- C1: renamed from C3; value 330 μF -> 100 μF; footprint Capacitor_SMD:CP_Elec_8x10 -> Capacitor_SMD:CP_Elec_5x5.8
- C17: renamed from C7; footprint Capacitor_SMD:C_0603_1608Metric -> Capacitor_SMD:C_0402_1005Metric
- C2: renamed from C4; value 1 μF -> 10 μF; footprint Capacitor_SMD:C_1206_3216Metric -> Capacitor_SMD:C_0805_2012Metric
- J8: renamed from J3; value Barrel_Jack_Switch -> Barrel_JACK
- R10: renamed from R3; footprint Resistor_SMD:R_0603_1608Metric -> Resistor_SMD:R_0402_1005Metric
- R11: renamed from R4; footprint Resistor_SMD:R_0603_1608Metric -> Resistor_SMD:R_0402_1005Metric
- R5, R6: value 10 kΩ -> 39 Ω; footprint Resistor_SMD:R_0603_1608Metric -> Resistor_SMD:R_0402_1005Metric
- R7: renamed from R1; footprint Resistor_SMD:R_0603_1608Metric -> Resistor_SMD:R_0402_1005Metric
- R8: renamed from R2; footprint Resistor_SMD:R_0603_1608Metric -> Resistor_SMD:R_0402_1005Metric
- R9: renamed from R10; footprint Resistor_SMD:R_0603_1608Metric -> Resistor_SMD:R_0402_1005Metric
- renumbered D6 to D2, D2 to D3, D3 to D4, J4 to J9, U4 to U3, U3 to U6
Connections:
- net labels added: A4, A5, A6, D1, D10, D4, D5, D8, D9, RST, SWCLK, SWDIO, USB_ID, nRF_EN, nRF_PWR, nRF_RST, nRF_STAT, nRF_SWCLK, nRF_SWDIO, nRF_SW_EN
- net labels removed: AND_RX, AND_TX, NETLIGHT, ONOFF_PIN, PWR_STAT, RTC_I, TLL_RST, TLL_RX, TLL_TX, TTL_3.3V, V_1.8
- wire segments 78 -> 188
- no-connect marks 47 -> 41
Other:
- note added: "Debug LEDs"
- note added: "NFC"
- note removed: "AND gate (Debug mode enable)"
- note removed: "MS5803 On-Board Pressure Sensor"
- note removed: "RFID"
- note removed: "RTC\n"
- note removed: "SIM 7000"
- note removed: "USB-TTL Converter\n"
- moved on the sheet: AE1, AT1, AT2, C1, C17, D2, D3, D4, G1, H1, H2, I1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

Commit message: added battery connector
Parts:
- removed C8: 100 nF, Capacitor_SMD:C_0402_1005Metric, symbol Device:C_Small
- removed J8: Barrel_JACK, Connector_BarrelJack:BarrelJack_Horizontal, symbol Connector:Barrel_Jack_Switch
- removed R15: 10 kΩ, Resistor_SMD:R_0402_1005Metric, symbol Device:R
- added J8: Jack-DC, Connector_JST:JST_PH_S2B-PH-SM4-TB_1x02-1MP_P2.00mm_Horizontal, symbol Connector:Jack-DC
- added U7, U8: MAX40203ANS, Package_BGA:WLP-4_0.73x0.73mm_Layout2x2_P0.35mm_Ball0.22mm_Pad0.2mm_NSMD, symbol Analog_Switch:MAX40200ANS
- J4, J5: footprint SIMFootprints:TC2030 -> SIMFootprints:TC2030_Pinless
- R14: value 10 kΩ -> 18 kΩ
- U4: footprint (none) -> SIMFootprints:nRF9160
Connections:
- net GND is gone; now on net -BATT: AT1.2, AT2.2, C1.2, C10.1, C11.2, C12.2, C13.2, C14.1, C15.1, C16.1, C17.1, C18.1, C2.2, C3.2, C4.2, C5.1, C6.2, C7.2, C9.2, I1.4 (GND), J1.6 (VSS), J1.9 (SHIELD), J3.3 (Pin_3), J3.4 (Pin_4), J4.5 (Pin_5), J5.5 (Pin_5), J7.2 (Pin_2), J9.5 (GND), R10.2, R11.2, R9.2, SW1.1, U1.1 (GND), U2.18 (GND), U2.35 (GND), U2.42 (GND), U2.5 (GNDANA), U3.2 (VSS), U4.1 (GND_Shield), U4.103 (VSS), U4.11 (GND_Shield), U4.14 (GND_Shield), U4.17 (GND_Shield), U4.21 (GND_Shield), U4.27 (GND_Shield), U4.31 (GND_Shield), U4.36 (GND_Shield), U4.41 (GND_Shield), U4.44 (GND_Shield), U4.47 (GND_Shield), U4.5 (GND_Shield), U4.50 (GND_Shield), U4.52 (GND_Shield), U4.56 (GND_Shield), U4.6 (GND_Shield), U4.60 (GND_Shield), U4.62 (GND_Shield), U4.63 (GND_Shield), U4.65 (GND_Shield), U4.66 (GND_Shield), U4.68 (GND_Shield), U4.69 (GND_Shield), U4.7 (GND_Shield), U4.72 (GND_Shield), U4.74 (GND_Shield), U4.75 (GND_Shield), U4.76 (GND_Shield), U4.77 (GND_Shield), U4.78 (GND_Shield), U4.79 (GND_Shield), U4.8 (GND_Shield), U4.80 (GND_Shield), U4.81 (GND_Shield), U4.82 (GND_Shield), U4.85 (GND_Shield), U4.9 (GND_Shield), U4.90 (GND_Shield), U4.94 (GND_Shield), U4.98 (GND_Shield), U5.1 (G), U5.4 (G), U6.2
- net USB_V: now also U7.A1 (VDD), U7.B1 (EN)
- net VNFC: now also R8.1
- net VPP: now also U7.A2 (OUT), U8.A2 (OUT)
- net V_3.3: no longer R8.1
- net nRF_PWR: now also U4.83 (P0.26); no longer U4.4 (P0.07)
- net nRF_STAT: now also U4.84 (P0.27); no longer U4.3 (P0.06)
- net -BATT: now reaches R14.2
- net -BATT: now also J8.2, U7.B2 (GND), U8.B2 (GND)
- new net +BATT: J8.1, U8.A1 (VDD), U8.B1 (EN)
- no-connect marks 41 -> 42
Changed lines of the file:
@@
 SCL
-$Comp
-L power:VPP #PWR019
-U 1 1 5CE71F49
-P 5000 1100
-F 0 "#PWR019" H 5000 950 50  0001 C CNN
-F 1 "VPP" H 5000 1250 50  0000 C CNN
-F 2 "" H 5000 1100 50  0000 C CNN
-F 3 "" H 5000 1100 50  0000 C CNN
-	1    5000 1100
-	0    1    1    0
-$EndComp
-$Comp
-L power:GND #PWR020
-U 1 1 5CE71F8D
-P 5000 1200
-F 0 "#PWR020" H 5000 950 50  0001 C CNN
-F 1 "GND" H 5000 1050 50  0000 C CNN
-F 2 "" H 5000 1200 50  0000 C CNN
-F 3 "" H 5000 1200 50  0000 C CNN
-	1    5000 1200
-	0    -1   -1   0
-$EndComp
 $Comp
 L power:GND #PWR021
 U 1 1 5CE71FD1
-P 5000 1300
-F 0 "#PWR021" H 5000 1050 50  0001 C CNN
-F 1 "GND" H 5000 1150 50  0000 C CNN
-F 2 "" H 5000 1300 50  0000 C CNN
-F 3 "" H 5000 1300 50  0000 C CNN
-	1    5000 1300
-	0    -1   -1   0
+P 5300 1350
+F 0 "#PWR021" H 5300 1100 50  0001 C CNN
+F 1 "GND" H 5300 1200 50  0000 C CNN
+F 2 "" H 5300 1350 50  0000 C CNN
+F 3 "" H 5300 1350 50  0000 C CNN
+	1    5300 1350
+	1    0    0    -1
 $EndComp
 $Comp
@@
 	-1   0    0    1
 $EndComp
-Text GLabel 7550 1600 3    60   Input ~ 0
-V_3.3
 Wire Wire Line
 	7450 1300 7550 1300
@@
 ATmega RST
 $Comp
-L Connector:Barrel_Jack_Switch J8
-U 1 1 5FE17CB9
-P 4700 1200
-F 0 "J8" H 4757 1517 50  0000 C CNN
-F 1 "Barrel_JACK" H 4757 1426 50  0000 C CNN
-F 2 "Connector_BarrelJack:BarrelJack_Horizontal" H 4750 1160 50  0001 C CNN
-F 3 "~" H 4750 1160 50  0001 C CNN
-	1    4700 1200
-	1    0    0    -1
-$EndComp
-$Comp
 L SIM7000-rescue:SPST-simcom SW1
 U 1 1 5D0B2067
@@
 $EndComp
 $Comp
-L Device:C_Small C8
-U 1 1 5FD91999
-P 6150 2750
-F 0 "C8" V 5921 2750 50  0000 C CNN
-F 1 "100 nF" V 6012 2750 50  0000 C CNN
-F 2 "Capacitor_SMD:C_0402_1005Metric" H 6150 2750 50  0001 C CNN
-F 3 "~" H 6150 2750 50  0001 C CNN
-	1    6150 2750
-	0    1    1    0
-$EndComp
-$Comp
 L Device:C_Small C7
 U 1 1 5FD91F72
@@
 	6300 2850 6300 2400
 Wire Wire Line
-	6400 2850 6400 2750
-Wire Wire Line
 	6700 2450 6800 2450
 Connection ~ 6700 2450
@@
 Wire Wire Line
 	6300 2400 6300 2300
-Wire Wire Line
-	6400 2750 6250 2750
-Connection ~ 6400 2750
-Wire Wire Line
-	6400 2750 6400 2300
 $Comp
 L power:GND #PWR028
@@
 F 3 "" H 6050 2400 50  0001 C CNN
 	1    6050 2400
-	0    1    1    0
-$EndComp
-$Comp
-L power:GND #PWR023
-U 1 1 5FDA2FD6
-P 6050 2750
-F 0 "#PWR023" H 6050 2500 50  0001 C CNN
-F 1 "GND" V 6055 2622 50  0000 R CNN
-F 2 "" H 6050 2750 50  0001 C CNN
-F 3 "" H 6050 2750 50  0001 C CNN
-	1    6050 2750
 	0    1    1    0
 $EndComp
@@
 F 0 "J4" H 2550 4717 50  0000 C CNN
 F 1 "SAMD_DBG" H 2550 4626 50  0000 C CNN
-F 2 "SIMFootprints:TC2030" H 2500 4400 50  0001 C CNN
+F 2 "SIMFootprints:TC2030_Pinless" H 2500 4400 50  0001 C CNN
 F 3 "~" H 2500 4400 50  0001 C CNN
 	1    2500 4400
@@
 F 0 "U4" H 10400 4300 60  0000 C CNN
 F 1 "NRF9160" H 10400 4200 60  0000 C CNN
-F 2 "" H 10400 4100 60  0001 C CNN
+F 2 "SIMFootprints:nRF9160" H 10400 4100 60  0001 C CNN
 F 3 "" H 10400 4100 60  0001 C CNN
 	1    10400 3950
@@
 F 0 "U4" H 15050 4850 60  0000 C CNN
 F 1 "NRF9160" H 15050 4750 60  0000 C CNN
-F 2 "" H 15000 4450 60  0001 C CNN
+F 2 "SIMFootprints:nRF9160" H 15000 4450 60  0001 C CNN
 F 3 "" H 15000 4450 60  0001 C CNN
 	2    15000 4300
@@
 F 0 "J5" H 2550 5917 50  0000 C CNN
 F 1 "nRF_DBG" H 2550 5826 50  0000 C CNN
-F 2 "SIMFootprints:TC2030" H 2500 5600 50  0001 C CNN
+F 2 "SIMFootprints:TC2030_Pinless" H 2500 5600 50  0001 C CNN
 F 3 "~" H 2500 5600 50  0001 C CNN
 	1    2500 5600
@@
 NoConn ~ 9700 6050
 NoConn ~ 9700 5950
-NoConn ~ 9700 5850
-NoConn ~ 9700 5750
 NoConn ~ 9700 5650
 NoConn ~ 9700 5550
@@
 Wire Wire Line
 	10150 1550 10200 1550
-Text GLabel 9700 3750 0    60   Input ~ 0
+Text GLabel 9700 5850 0    60   Input ~ 0
 nRF_STAT
-Text GLabel 9700 3850 0    60   Input ~ 0
+Text GLabel 9700 5750 0    60   Input ~ 0
 nRF_PWR
 NoConn ~ 9700 4450
@@
 P 8900 4100
 F 0 "R14" H 8970 4146 50  0000 L CNN
-F 1 "10 kΩ" H 8970 4055 50  0000 L CNN
+F 1 "18 kΩ" H 8970 4055 50  0000 L CNN
 F 2 "Resistor_SMD:R_0402_1005Metric" V 8830 4100 50  0001 C CNN
 F 3 "~" H 8900 4100 50  0001 C CNN
@@
 L power:GND #PWR042
 U 1 1 605FF3CD
-P 8900 4600
-F 0 "#PWR042" H 8900 4350 50  0001 C CNN
-F 1 "GND" H 8900 4450 50  0000 C CNN
-F 2 "" H 8900 4600 50  0000 C CNN
-F 3 "" H 8900 4600 50  0000 C CNN
-	1    8900 4600
+P 8900 4250
+F 0 "#PWR042" H 8900 4000 50  0001 C CNN
+F 1 "GND" H 8900 4100 50  0000 C CNN
+F 2 "" H 8900 4250 50  0000 C CNN
+F 3 "" H 8900 4250 50  0000 C CNN
+	1    8900 4250
 	1    0    0    -1
 $EndComp
 Wire Wire Line
 	8900 3600 8900 3650
-$Comp
-L Device:R R15
-U 1 1 60628742
-P 8900 4450
-F 0 "R15" H 8970 4496 50  0000 L CNN
-F 1 "10 kΩ" H 8970 4405 50  0000 L CNN
-F 2 "Resistor_SMD:R_0402_1005Metric" V 8830 4450 50  0001 C CNN
-F 3 "~" H 8900 4450 50  0001 C CNN
-	1    8900 4450
-	1    0    0    -1
-$EndComp
-Wire Wire Line
-	8900 4250 8900 4300
 $Comp
 L Device:Crystal_Small Y1
@@
 Connection ~ 4750 3050
 Connection ~ 4750 3250
+Text GLabel 7550 1600 3    60   Input ~ 0
+VNFC
+Wire Wire Line
+	6400 2300 6400 2850
+NoConn ~ 9700 3750
+NoConn ~ 9700 3850
+$Comp
+L Analog_Switch:MAX40200ANS U7
+U 1 1 601C01EE
+P 1900 9650
+F 0 "U7" H 1900 10017 50  0000 C CNN
+F 1 "MAX40203ANS" H 1900 9926 50  0000 C CNN
+F 2 "Package_BGA:WLP-4_0.73x0.73mm_Layout2x2_P0.35mm_Ball0.22mm_Pad0.2mm_NSMD" H 1900 10050 50  0001 C CNN
+F 3 "https://datasheets.maximintegrated.com/en/ds/MAX40200.pdf" H 1900 10050 50  0001 C CNN
+	1    1900 9650
+	1    0    0    -1
+$EndComp
+$Comp
+L Analog_Switch:MAX40200ANS U8
+U 1 1 601C2377
+P 1900 10600
+F 0 "U8" H 1900 10967 50  0000 C CNN
+F 1 "MAX40203ANS" H 1900 10876 50  0000 C CNN
+F 2 "Package_BGA:WLP-4_0.73x0.73mm_Layout2x2_P0.35mm_Ball0.22mm_Pad0.2mm_NSMD" H 1900 11000 50  0001 C CNN
+F 3 "https://datasheets.maximintegrated.com/en/ds/MAX40200.pdf" H 1900 11000 50  0001 C CNN
+	1    1900 10600
+	1    0    0    -1
+$EndComp
+$Comp
+L power:GND #PWR0101
+U 1 1 601C2825
+P 1900 9950
+F 0 "#PWR0101" H 1900 9700 50  0001 C CNN
+F 1 "GND" H 1905 9777 50  0000 C CNN
+F 2 "" H 1900 9950 50  0001 C CNN
+F 3 "" H 1900 9950 50  0001 C CNN
+	1    1900 9950
+	1    0    0    -1
+$EndComp
+$Comp
+L power:GND #PWR0102
+U 1 1 601C345F
+P 1900 10900
+F 0 "#PWR0102" H 1900 10650 50  0001 C CNN
+F 1 "GND" H 1905 10727 50  0000 C CNN
+F 2 "" H 1900 10900 50  0001 C CNN
+F 3 "" H 1900 10900 50  0001 C CNN
+	1    1900 10900
+	1    0    0    -1
+$EndComp
+$Comp
+L power:VPP #PWR0103
+U 1 1 601C377D
+P 2750 10150
+F 0 "#PWR0103" H 2750 10000 50  0001 C CNN
+F 1 "VPP" H 2750 10300 50  0000 C CNN
+F 2 "" H 2750 10150 50  0000 C CNN
+F 3 "" H 2750 10150 50  0000 C CNN
+	1    2750 10150
+	0    1    1    0
+$EndComp
+Wire Wire Line
+	2300 9550 2500 9550
+Wire Wire Line
+	2500 9550 2500 10150
+Wire Wire Line
+	2500 10150 2750 10150
+Wire Wire Line
+	2300 10500 2500 10500
+Wire Wire Line
+	2500 10500 2500 10150
+Connection ~ 2500 10150
+$Comp
+L power:+BATT #PWR0104
+U 1 1 601DB601
+P 5000 1100
+F 0 "#PWR0104" H 5000 950 50  0001 C CNN
+F 1 "+BATT" V 5015 1228 50  0000 L CNN
+F 2 "" H 5000 1100 50  0001 C CNN
+F 3 "" H 5000 1100 50  0001 C CNN
+	1    5000 1100
+	0    1    1    0
+$EndComp
+$Comp
+L power:+BATT #PWR0105
+U 1 1 601DC315
+P 1300 10500
+F 0 "#PWR0105" H 1300 10350 50  0001 C CNN
+F 1 "+BATT" V 1315 10627 50  0000 L CNN
+F 2 "" H 1300 10500 50  0001 C CNN
+F 3 "" H 1300 10500 50  0001 C CNN
+	1    1300 10500
+	0    -1   -1   0
+$EndComp
+Wire Wire Line
+	1300 10500 1400 10500
+Wire Wire Line
+	1500 10700 1400 10700
+Wire Wire Line
+	1400 10700 1400 10500
+Connection ~ 1400 10500
+Wire Wire Line
+	1400 10500 1500 10500
+Text GLabel 1300 9550 0    60   Input ~ 0
+USB_V
+Wire Wire Line
+	1300 9550 1400 9550
+Wire Wire Line
+	1500 9750 1400 9750
+Wire Wire Line
+	1400 9750 1400 9550
+Connection ~ 1400 9550
+Wire Wire Line
+	1400 9550 1500 9550
+$Comp
+L Connector:Jack-DC J8
+U 1 1 6025265A
+P 4700 1200
+F 0 "J8" H 4757 1525 50  0000 C CNN
+F 1 "Jack-DC" H 4757 1434 50  0000 C CNN
+F 2 "Connector_JST:JST_PH_S2B-PH-SM4-TB_1x02-1MP_P2.00mm_Horizontal" H 4750 1160 50  0001 C CNN
+F 3 "~" H 4750 1160 50  0001 C CNN
+	1    4700 1200
+	1    0    0    -1
+$EndComp
+$Comp
+L power:-BATT #PWR0106
+U 1 1 60253242
+P 5100 1350
+F 0 "#PWR0106" H 5100 1200 50  0001 C CNN
+F 1 "-BATT" H 5115 1523 50  0000 C CNN
+F 2 "" H 5100 1350 50  0001 C CNN
+F 3 "" H 5100 1350 50  0001 C CNN
+	1    5100 1350
+	-1   0    0    1
+$EndComp
+Wire Wire Line
+	5000 1300 5100 1300
+Wire Wire Line
+	5300 1300 5300 1350
+Wire Wire Line
+	5100 1350 5100 1300
+Connection ~ 5100 1300
+Wire Wire Line
+	5100 1300 5300 1300
+NoConn ~ 13250 1050
 $EndSCHEMATC

Commit message: changed connectivity
Parts:
- J6: footprint Connector_PinHeader_2.54mm:PinHeader_1x10_P2.54mm_Vertical -> Connector_PinSocket_1.27mm:PinSocket_1x10_P1.27mm_Vertical
Changed lines of the file:
@@
 F 0 "J6" H 2980 6642 50  0000 L CNN
 F 1 "Conn_01x10" H 2980 6551 50  0000 L CNN
-F 2 "Connector_PinHeader_2.54mm:PinHeader_1x10_P2.54mm_Vertical" H 2900 6650 50  0001 C CNN
+F 2 "Connector_PinSocket_1.27mm:PinSocket_1x10_P1.27mm_Vertical" H 2900 6650 50  0001 C CNN
 F 3 "~" H 2900 6650 50  0001 C CNN
 	1    2900 6650
