File: nano/EDA/EDA/BoSLnano.sch (KiCad schematic (older format))
At the start: 63 parts, among them J1 Micro_SD_Card, J2 Conn_01x07, J3 Conn_01x04, J4 SAMD_DBG, J5 nRF_DBG, J6 Conn_01x10, J7 Conn_01x04, J8 Jack-DC, J9 USB_B_Micro, SW1 SPST, U1 MCP1700-3302E_SOT23, U2 ATSAMD21G18A-MUT, U3 NT3H2111W0FTT, U4 NRF9160, U5 BGA524N6, U6 MSQA6V1W5T2G, U7 MAX40203ANS, U8 MAX40203ANS, Y1 32.768kHz

Commit message: modifed nano
Parts:
- removed H1, H2: MountingHole, MountingHole:MountingHole_2.2mm_M2_Pad, symbol Mechanical:MountingHole
- added D?: LED, LED_SMD:LED_0603_1608Metric, symbol Device:LED
- added R?: 3.3 kΩ, Resistor_SMD:R_0402_1005Metric, symbol Device:R
Connections:
- net -BATT: now also D2.1 (K), D3.1 (K), D4.1 (K), D?.1 (K); no longer R10.2, R11.2, R9.2
- net D1: no longer U2.32 (PA23)
- net NFC_I: now also U2.32 (PA23); no longer U2.31 (PA22)
- net USB_V: now also R9.1; no longer D2.2 (A)
- net VNFC: now also U2.31 (PA22); no longer U2.7 (PB08)
- net nRF_PWR: now also R11.1; no longer D4.2 (A)
- net nRF_STAT: now also R10.1; no longer D3.2 (A)
- net at R13.2, R14.1: now also U4.42 (P0.25_TRACEDATA3); no longer U4.15 (P0.08)
- new net: D2.2 (A), R9.2
- new net: D4.2 (A), R11.2
- new net: D3.2 (A), R10.2
- new net: R?.1, U2.7 (PB08)
- new net: D?.2 (A), R?.2
- no-connect marks 42 -> 41
Other:
- note removed: "Mounting Holes\n"
- moved on the sheet: D2, D3, D4, R10, R11, R13, R14, R9
Changed lines of the file:
@@
 L Device:LED D4
 U 1 1 5D4315A4
+P 10800 1550
+F 0 "D4" H 10800 1650 50  0000 C CNN
+F 1 "LED" H 10800 1450 50  0000 C CNN
+F 2 "LED_SMD:LED_0603_1608Metric" H 10800 1550 50  0001 C CNN
+F 3 "" H 10800 1550 50  0000 C CNN
+	1    10800 1550
+	-1   0    0    1
+$EndComp
+$Comp
+L Device:R R11
+U 1 1 5D4315AA
 P 10350 1550
-F 0 "D4" H 10350 1650 50  0000 C CNN
-F 1 "LED" H 10350 1450 50  0000 C CNN
-F 2 "LED_SMD:LED_0603_1608Metric" H 10350 1550 50  0001 C CNN
+F 0 "R11" V 10250 1550 50  0000 C CNN
+F 1 "3.3 kΩ" V 10450 1550 50  0000 C CNN
+F 2 "Resistor_SMD:R_0402_1005Metric" V 10280 1550 50  0001 C CNN
 F 3 "" H 10350 1550 50  0000 C CNN
 	1    10350 1550
-	-1   0    0    1
-$EndComp
-$Comp
-L Device:R R11
-U 1 1 5D4315AA
-P 10800 1550
-F 0 "R11" V 10700 1550 50  0000 C CNN
-F 1 "3.3 kΩ" V 10900 1550 50  0000 C CNN
-F 2 "Resistor_SMD:R_0402_1005Metric" V 10730 1550 50  0001 C CNN
-F 3 "" H 10800 1550 50  0000 C CNN
-	1    10800 1550
 	0    -1   -1   0
 $EndComp
@@
 L Device:LED D3
 U 1 1 5D432F55
+P 10800 1250
+F 0 "D3" H 10800 1350 50  0000 C CNN
+F 1 "LED" H 10800 1150 50  0000 C CNN
+F 2 "LED_SMD:LED_0603_1608Metric" H 10800 1250 50  0001 C CNN
+F 3 "" H 10800 1250 50  0000 C CNN
+	1    10800 1250
+	-1   0    0    1
+$EndComp
+$Comp
+L Device:R R10
+U 1 1 5D432F5B
 P 10350 1250
-F 0 "D3" H 10350 1350 50  0000 C CNN
-F 1 "LED" H 10350 1150 50  0000 C CNN
-F 2 "LED_SMD:LED_0603_1608Metric" H 10350 1250 50  0001 C CNN
+F 0 "R10" V 10450 1250 50  0000 C CNN
+F 1 "3.3 kΩ" V 10250 1250 50  0000 C CNN
+F 2 "Resistor_SMD:R_0402_1005Metric" V 10280 1250 50  0001 C CNN
 F 3 "" H 10350 1250 50  0000 C CNN
 	1    10350 1250
-	-1   0    0    1
-$EndComp
-$Comp
-L Device:R R10
-U 1 1 5D432F5B
-P 10800 1250
-F 0 "R10" V 10900 1250 50  0000 C CNN
-F 1 "3.3 kΩ" V 10700 1250 50  0000 C CNN
-F 2 "Resistor_SMD:R_0402_1005Metric" V 10730 1250 50  0001 C CNN
-F 3 "" H 10800 1250 50  0000 C CNN
-	1    10800 1250
 	0    -1   -1   0
 $EndComp
@@
 	500  3750 500  10500
 $Comp
-L Mechanical:MountingHole H1
-U 1 1 5D620C83
-P 14750 850
-F 0 "H1" H 14850 896 50  0000 L CNN
-F 1 "MountingHole" H 14850 805 50  0000 L CNN
-F 2 "MountingHole:MountingHole_2.2mm_M2_Pad" H 14750 850 50  0001 C CNN
-F 3 "~" H 14750 850 50  0001 C CNN
-	1    14750 850
-	1    0    0    -1
-$EndComp
-$Comp
-L Mechanical:MountingHole H2
-U 1 1 5D622088
-P 14750 1100
-F 0 "H2" H 14850 1146 50  0000 L CNN
-F 1 "MountingHole" H 14850 1055 50  0000 L CNN
-F 2 "MountingHole:MountingHole_2.2mm_M2_Pad" H 14750 1100 50  0001 C CNN
-F 3 "~" H 14750 1100 50  0001 C CNN
-	1    14750 1100
-	1    0    0    -1
-$EndComp
-Text Notes 14400 700  0    60   ~ 0
-Mounting Holes\n
-$Comp
 L SIM7000-rescue:AT-ant AT2
 U 1 1 5DBBFC5D
@@
 Text GLabel 7100 900  1    60   Input ~ 0
 VNFC
-Text GLabel 7500 3350 2    60   Input ~ 0
+Text GLabel 5500 5350 0    60   Input ~ 0
 VNFC
 NoConn ~ 6900 900
@@
 Text GLabel 7650 1300 2    60   Input ~ 0
 NFC_I
-Text GLabel 5500 5350 0    60   Input ~ 0
+Text GLabel 5500 5450 0    60   Input ~ 0
 NFC_I
 $Comp
@@
 Text GLabel 2000 4100 1    60   Input ~ 0
 V_3.3
-$Comp
-L SIM7000-rescue:NRF9160 U4
-U 1 1 5FEB3BD7
-P 10400 3950
-F 0 "U4" H 10400 4300 60  0000 C CNN
-F 1 "NRF9160" H 10400 4200 60  0000 C CNN
-F 2 "SIMFootprints:nRF9160" H 10400 4100 60  0001 C CNN
-F 3 "" H 10400 4100 60  0001 C CNN
-	1    10400 3950
-	1    0    0    -1
-$EndComp
 Wire Wire Line
 	14250 2800 14100 2800
@@
 Text GLabel 5500 3450 0    60   Input ~ 0
 AREF
-Text GLabel 5500 5450 0    60   Input ~ 0
-D1
 Text GLabel 5500 4150 0    60   Input ~ 0
 D2
@@
 NoConn ~ 9700 6050
 NoConn ~ 9700 5950
-NoConn ~ 9700 5650
 NoConn ~ 9700 5550
 NoConn ~ 9700 5450
@@
 L Device:LED D2
 U 1 1 5D430CC2
+P 10800 950
+F 0 "D2" H 10800 1050 50  0000 C CNN
+F 1 "LED" H 10800 850 50  0000 C CNN
+F 2 "LED_SMD:LED_0603_1608Metric" H 10800 950 50  0001 C CNN
+F 3 "" H 10800 950 50  0000 C CNN
+	1    10800 950
+	-1   0    0    1
+$EndComp
+Wire Wire Line
+	10150 950  10200 950
+$Comp
+L Device:R R9
+U 1 1 5D430D8C
 P 10350 950
-F 0 "D2" H 10350 1050 50  0000 C CNN
-F 1 "LED" H 10350 850 50  0000 C CNN
-F 2 "LED_SMD:LED_0603_1608Metric" H 10350 950 50  0001 C CNN
+F 0 "R9" V 10430 950 50  0000 C CNN
+F 1 "3.3 kΩ" V 10250 950 50  0000 C CNN
+F 2 "Resistor_SMD:R_0402_1005Metric" V 10280 950 50  0001 C CNN
 F 3 "" H 10350 950 50  0000 C CNN
 	1    10350 950
-	-1   0    0    1
-$EndComp
-Wire Wire Line
-	10150 950  10200 950
-$Comp
-L Device:R R9
-U 1 1 5D430D8C
-P 10800 950
-F 0 "R9" V 10880 950 50  0000 C CNN
-F 1 "3.3 kΩ" V 10700 950 50  0000 C CNN
-F 2 "Resistor_SMD:R_0402_1005Metric" V 10730 950 50  0001 C CNN
-F 3 "" H 10800 950 50  0000 C CNN
-	1    10800 950
 	0    -1   -1   0
 $EndComp
@@
 NoConn ~ 9700 4450
 Wire Wire Line
-	9700 3950 8900 3950
+	9700 5650 8900 5650
 $Comp
 L Device:R R14
 U 1 1 605F45E5
-P 8900 4100
-F 0 "R14" H 8970 4146 50  0000 L CNN
-F 1 "18 kΩ" H 8970 4055 50  0000 L CNN
-F 2 "Resistor_SMD:R_0402_1005Metric" V 8830 4100 50  0001 C CNN
-F 3 "~" H 8900 4100 50  0001 C CNN
-	1    8900 4100
+P 8900 5800
+F 0 "R14" H 8970 5846 50  0000 L CNN
+F 1 "18 kΩ" H 8970 5755 50  0000 L CNN
+F 2 "Resistor_SMD:R_0402_1005Metric" V 8830 5800 50  0001 C CNN
+F 3 "~" H 8900 5800 50  0001 C CNN
+	1    8900 5800
 	1    0    0    -1
 $EndComp
@@
 L Device:R R13
 U 1 1 605F54CB
-P 8900 3800
-F 0 "R13" H 8970 3846 50  0000 L CNN
-F 1 "10 kΩ" H 8970 3755 50  0000 L CNN
-F 2 "Resistor_SMD:R_0402_1005Metric" V 8830 3800 50  0001 C CNN
-F 3 "~" H 8900 3800 50  0001 C CNN
-	1    8900 3800
-	1    0    0    -1
-$EndComp
-Connection ~ 8900 3950
-Text GLabel 8900 3600 1    60   Input ~ 0
+P 8900 5500
+F 0 "R13" H 8970 5546 50  0000 L CNN
+F 1 "10 kΩ" H 8970 5455 50  0000 L CNN
+F 2 "Resistor_SMD:R_0402_1005Metric" V 8830 5500 50  0001 C CNN
+F 3 "~" H 8900 5500 50  0001 C CNN
+	1    8900 5500
+	1    0    0    -1
+$EndComp
+Connection ~ 8900 5650
+Text GLabel 8900 5300 1    60   Input ~ 0
 USB_V
 $Comp
 L power:GND #PWR042
 U 1 1 605FF3CD
-P 8900 4250
-F 0 "#PWR042" H 8900 4000 50  0001 C CNN
-F 1 "GND" H 8900 4100 50  0000 C CNN
-F 2 "" H 8900 4250 50  0000 C CNN
-F 3 "" H 8900 4250 50  0000 C CNN
-	1    8900 4250
-	1    0    0    -1
-$EndComp
-Wire Wire Line
-	8900 3600 8900 3650
+P 8900 5950
+F 0 "#PWR042" H 8900 5700 50  0001 C CNN
+F 1 "GND" H 8900 5800 50  0000 C CNN
+F 2 "" H 8900 5950 50  0000 C CNN
+F 3 "" H 8900 5950 50  0000 C CNN
+	1    8900 5950
+	1    0    0    -1
+$EndComp
+Wire Wire Line
+	8900 5300 8900 5350
 $Comp
 L Device:Crystal_Small Y1
@@
 	5100 1300 5300 1300
 NoConn ~ 13250 1050
+$Comp
+L SIM7000-rescue:NRF9160 U4
+U 1 1 5FEB3BD7
+P 10400 3950
+F 0 "U4" H 10400 4300 60  0000 C CNN
+F 1 "NRF9160" H 10400 4200 60  0000 C CNN
+F 2 "SIMFootprints:nRF9160" H 10400 4100 60  0001 C CNN
+F 3 "" H 10400 4100 60  0001 C CNN
+	1    10400 3950
+	1    0    0    -1
+$EndComp
+$Comp
+L Device:LED D?
+U 1 1 601A9F02
+P 8500 3350
+F 0 "D?" H 8500 3450 50  0000 C CNN
+F 1 "LED" H 8500 3250 50  0000 C CNN
+F 2 "LED_SMD:LED_0603_1608Metric" H 8500 3350 50  0001 C CNN
+F 3 "" H 8500 3350 50  0000 C CNN
+	1    8500 3350
+	-1   0    0    1
+$EndComp
+$Comp
+L Device:R R?
+U 1 1 601A9F08
+P 8050 3350
+F 0 "R?" V 7950 3350 50  0000 C CNN
+F 1 "3.3 kΩ" V 8150 3350 50  0000 C CNN
+F 2 "Resistor_SMD:R_0402_1005Metric" V 7980 3350 50  0001 C CNN
+F 3 "" H 8050 3350 50  0000 C CNN
+	1    8050 3350
+	0    -1   -1   0
+$EndComp
+$Comp
+L power:GND #PWR?
+U 1 1 601A9F0E
+P 8750 3450
+F 0 "#PWR?" H 8750 3200 50  0001 C CNN
+F 1 "GND" H 8750 3300 50  0000 C CNN
+F 2 "" H 8750 3450 50  0000 C CNN
+F 3 "" H 8750 3450 50  0000 C CNN
+	1    8750 3450
+	1    0    0    -1
+$EndComp
+Wire Wire Line
+	8200 3350 8350 3350
+Wire Wire Line
+	7900 3350 7500 3350
+Wire Wire Line
+	8650 3350 8750 3350
+Wire Wire Line
+	8750 3350 8750 3450
 $EndSCHEMATC
