File: nano/EDA/EDA/_autosave-BoSLnano.sch (KiCad schematic (older format))
At the start: 66 parts, among them J1 Micro_SD_Card, J2 Conn_01x07, J3 Conn_01x04, J4 SAMD_DBG, J5 nRF_DBG, J6 Conn_01x10, J7 Conn_01x04, J8 Jack-DC, J9 USB_B_Micro, SW1 SPST, U1 MCP1700-3302E_SOT23, U2 ATSAMD21G18A-MUT, U3 NT3H2111W0FTT, U4 NRF9160, U5 BGA524N6, U6 MSQA6V1W5T2G, U7 MAX40203ANS, U8 MAX40203ANS, Y1 32.768kHz

Commit message: made to be 70 mm
Parts:
- removed J6: Conn_01x10, Connector_PinSocket_1.27mm:PinSocket_1x10_P1.27mm_Vertical, symbol Connector_Generic:Conn_01x10
- added J6: Conn_01x09, Connector_PinHeader_1.27mm:PinHeader_1x09_P1.27mm_Vertical, symbol Connector_Generic:Conn_01x09
- gave numbers to parts that had none: 5
- renumbered C9 to C8, C10 to C9, D2 to D3, D3 to D4, D4 to D5, J9 to J10, I1 to J9, R13 to R12, R14 to R13, R9 to R14, R10 to R15, R11 to R16, R12 to R17, U7 to U1, U8 to U2, U1 to U3, U2 to U4, U3 to U5, U4 to U6, U5 to U7, U6 to U8
Connections:
- net labels removed: D1
