File: micro/EDA/EDA/microBoSL.sch (KiCad schematic (older format))
At the start: 38 parts, among them J1 Conn_01x04, J2 Conn_02x03_Odd_Even, J3 Conn_01x04, J4 Conn_01x04, J5 Conn_01x02, J6 Conn_01x10, J7 Conn_01x02, J8 USB_B_Micro, Q1 DMG2302UK, SW1 PTS636 SM43J SMTR LFS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

Commit message: finished micro bosl design
Parts:
- removed G1: BoSL_Graphic, SIMFootprints:BoSL_Graphic, symbol SIM7000-rescue:BoSL_Graphic
Other:
- note added: "HEATSINK_GROUND"
- note removed: "HEATSINC_GROUND"
- moved on the sheet: C2, C3, C4, C5, D3, J1, J2, J3, J4, J6, J7, R1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

Commit message: changed some labled on microBoSL
Other:
- note added: "MCU"
- note added: "Motor MOSFET"
- note added: "USB-TTL Converter"
- moved on the sheet: C2, C3, C4, C5, J1, J2, J3, J4, J5, J6, J7, R1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

Commit message: added hardware documentation
Parts:
- J8: symbol Connector:USB_B_Micro -> microBoSL-rescue:USB_B_Micro-Connector
Changed lines of the file:
@@
 TLL_RX
 $Comp
-L Connector:USB_B_Micro J8
+L microBoSL-rescue:USB_B_Micro-Connector J8
 U 1 1 5D612C02
 P 14700 3950

Commit message: updated microbosl schematic
Parts:
- removed Q1: DMG2302UK, Package_TO_SOT_SMD:SOT-23, symbol Device:Q_NMOS_GSD
- removed R2: 1 kΩ, Resistor_SMD:R_0402_1005Metric, symbol Device:R
- removed U1, U2: MAX40200ANS, Package_BGA:WLP-4_0.73x0.73mm_Layout2x2_P0.35mm_Ball0.22mm_Pad0.2mm_NSMD, symbol Analog_Switch:MAX40200ANS
- removed U3: MCP1700-3302E_SOT23, Package_TO_SOT_SMD:SOT-23, symbol Regulator_Linear:MCP1700-3302E_SOT23
- removed U4: ATmega328-MMH, Package_DFN_QFN:QFN-28-1EP_4x4mm_P0.45mm_EP2.4x2.4mm, symbol MCU_Microchip_ATmega:ATmega328-MMH
- added C?: 1 μF, Capacitor_SMD:C_1206_3216Metric, symbol Device:C
- added C? (x3): 100 nF, Capacitor_SMD:C_0603_1608Metric, symbol Device:C
- added Q?: DMP2165UW, Package_TO_SOT_SMD:SOT-323_SC-70, symbol microBoSL-rescue:DMP2165UW
- added R? (x2): 4.7 MΩ, Capacitor_SMD:C_0402_1005Metric, symbol Device:R
- added R?: 10 kΩ, Resistor_SMD:R_0402_1005Metric, symbol Device:R
- added SW?: AYZ0103AGRLC, SIMFootprints:AYZ0103AGRLC, symbol microBoSL-rescue:AYZ0103AGRLC
- added U? (x2): TPS709A33DBVT, Package_TO_SOT_SMD:SOT-23-5, symbol microBoSL-rescue:TPS709A33DBVT
- added U?: ZXBM5210-S, Package_SO:SOIC-8_3.9x4.9mm_P1.27mm, symbol Driver_Motor:ZXBM5210-S
- added U?: ATmega328P-MMH, Package_DFN_QFN:QFN-28-1EP_4x4mm_P0.45mm_EP2.4x2.4mm, symbol MCU_Microchip_ATmega:ATmega328P-MMH
- J5: value Conn_01x02 -> BATTERY CONN
- J7: value Conn_01x02 -> MOTOR_OUT
- SW1: value PTS636 SM43J SMTR LFS -> RST_JMPR; footprint SIMFootprints:PTS636 SM43J SMTR LFS -> Jumper:SolderJumper-2_P1.3mm_Open_RoundedPad1.0x1.5mm
Connections:
- net labels added: MFWD, MREV, VBAT
- net labels removed: MOSFET
- wire segments 42 -> 97
- no-connect marks 15 -> 19
Other:
- moved on the sheet: C1, C2, C3, C4, C5, C6, C7, D1, D2, D3, J7, R1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

Commit message: worked on micro BOM
Parts:
- removed C1: 1 μF, Capacitor_SMD:C_1206_3216Metric, symbol Device:C
- C1: renamed from C?; value 1 μF -> 2.2 μF; footprint Capacitor_SMD:C_1206_3216Metric -> Capacitor_SMD:C_0805_2012Metric; Supplier (none) -> https://au.mouser.com/ProductDetail/Samsung-Electro-Mechani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
- C10: renamed from C6; footprint Capacitor_SMD:C_0603_1608Metric -> Capacitor_SMD:C_0402_1005Metric; Supplier (none) -> https://au.mouser.com/ProductDetail/AVX/04026D104KAT2A?qs=s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
- C11: renamed from C7; footprint Capacitor_SMD:C_0603_1608Metric -> Capacitor_SMD:C_0402_1005Metric; Supplier (none) -> https://au.mouser.com/ProductDetail/AVX/04026D104KAT2A?qs=s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
- C3, C4, C7: renamed from C?; footprint Capacitor_SMD:C_0603_1608Metric -> Capacitor_SMD:C_0402_1005Metric; Supplier (none) -> https://au.mouser.com/ProductDetail/AVX/04026D104KAT2A?qs=s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
- C5: renamed from C3; value 22 pF -> 15 pF; Supplier (none) -> https://au.mouser.com/ProductDetail/KEMET/C0402C150J8HACTU?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
- C6: renamed from C2; value 22 pF -> 15 pF; Supplier (none) -> https://au.mouser.com/ProductDetail/KEMET/C0402C150J8HACTU?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
- C8: renamed from C5; value 12 pF -> 15 pF; Supplier (none) -> https://au.mouser.com/ProductDetail/KEMET/C0402C150J8HACTU?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
- C9: renamed from C4; value 12 pF -> 15 pF; Supplier (none) -> https://au.mouser.com/ProductDetail/KEMET/C0402C150J8HACTU?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
- D1: renamed from D3; Supplier (none) -> https://au.mouser.com/ProductDetail/Wurth-Elektronik/150060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
- D2: renamed from D1; Supplier (none) -> https://au.mouser.com/ProductDetail/Wurth-Elektronik/150060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
- D3: renamed from D2; Supplier (none) -> https://au.mouser.com/datasheet/2/445/150060YS55040-1714218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
- J8: Supplier (none) -> https://au.mouser.com/ProductDetail/Molex/105133-0001?qs=nm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
- Q1: renamed from Q?; Supplier (none) -> https://au.mouser.com/ProductDetail/Diodes-Incorporated/DMP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
- R1: renamed from R?; Supplier (none) -> https://au.mouser.com/ProductDetail/Vishay-Dale/CRCW040210K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
- R10: renamed from R8; Supplier (none) -> https://au.mouser.com/ProductDetail/Vishay-Dale/CRCW04023K3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
- R2: renamed from R1; Supplier (none) -> https://au.mouser.com/ProductDetail/Vishay-Dale/CRCW040210K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
- R3: renamed from R4; Supplier (none) -> https://au.mouser.com/ProductDetail/Vishay-Dale/CRCW040210K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
- R4: renamed from R3; Supplier (none) -> https://au.mouser.com/ProductDetail/Vishay-Dale/CRCW040210K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
- R5, R6: renamed from R?; Supplier (none) -> https://au.mouser.com/ProductDetail/Vishay-Dale/CRCW04024M7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
- R7: renamed from R5; Supplier (none) -> https://au.mouser.com/ProductDetail/Vishay-Dale/CRCW040210K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
- R8: renamed from R6; Supplier (none) -> https://au.mouser.com/ProductDetail/Vishay-Dale/CRCW04023K3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
- R9: renamed from R7; Supplier (none) -> https://au.mouser.com/ProductDetail/Vishay-Dale/CRCW04023K3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
- SW2: renamed from SW?; Supplier (none) -> https://au.mouser.com/ProductDetail/CK/AYZ0103AGRLC?qs=dJbz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
- U3: renamed from U?; Supplier (none) -> https://au.mouser.com/ProductDetail/Microchip-Technology-At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
- U4: renamed from U?; Supplier (none) -> https://au.mouser.com/ProductDetail/Diodes-Incorporated/ZXB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
- U5: renamed from U6; Supplier (none) -> https://au.mouser.com/ProductDetail/Nexperia/74HC126PW-Q100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
- U6: renamed from U5; Supplier (none) -> https://www.digikey.com.au/product-detail/en/MCP7940NT-I-MN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
- U7: Supplier (none) -> https://au.mouser.com/ProductDetail/FTDI/FT232RQ-REEL?qs=D1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
- Y1: footprint Crystal:Crystal_SMD_EuroQuartz_MT-4Pin_3.2x2.5mm -> Crystal:Crystal_SMD_5032-2Pin_5.0x3.2mm; Supplier (none) -> https://au.mouser.com/ProductDetail/Diodes-Incorporated/F90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
- Y2: footprint Crystal:Crystal_SMD_EuroQuartz_EQ161-2Pin_3.2x1.5mm -> Crystal:Crystal_SMD_2012-2Pin_2.0x1.2mm; Supplier (none) -> https://au.mouser.com/ProductDetail/IQD/LFXTAL050789Reel?qs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
- gave numbers to parts that had none: 2
- renumbered J3 to J2, J4 to J3, J5 to J4, J2 to J5

Commit message: microbosl layout finished TODO: optimise/silkscreen
Parts:
- removed J2: Conn_01x04, Connector_PinHeader_1.27mm:PinHeader_1x04_P1.27mm_Vertical, symbol Connector_Generic:Conn_01x04
- removed J6: Conn_01x10, Connector_PinHeader_1.27mm:PinHeader_1x10_P1.27mm_Vertical, symbol Connector_Generic:Conn_01x10
- added J2: Conn_01x03, Connector_PinHeader_1.27mm:PinHeader_1x03_P1.27mm_Vertical, symbol Connector_Generic:Conn_01x03
- added J6: Conn_01x04, Connector_PinHeader_1.27mm:PinHeader_1x04_P1.27mm_Vertical, symbol Connector_Generic:Conn_01x04
- J1: footprint Connector_PinHeader_2.54mm:PinHeader_1x04_P2.54mm_Vertical -> Connector_PinHeader_1.27mm:PinHeader_1x04_P1.27mm_Vertical
- Y1: symbol Device:Crystal_GND24 -> Device:Crystal
Connections:
- net D8 is gone; now on net MREV: U3.10 (PB0)
- net GND: no longer Y1.2, Y1.4
- net MREV: no longer U3.12 (PB2)
- net TLL_RST: now also J2.1 (Pin_1)
- net TLL_RX: now also J2.2 (Pin_2)
- net TLL_TX: now also J2.3 (Pin_3)
- net VBAT: now also J3.2 (Pin_2)
- net VPP: no longer J3.2 (Pin_2)
- net at C5.2, U3.5 (XTAL1/PB6): now also Y1.2; no longer Y1.3
- net D11 renamed MOSI
- net MOSI: now also J6.3 (Pin_3)
- net D12 renamed MISO
- net MISO: now also J6.2 (Pin_2)
- net D13 renamed SCLK
- net SCLK: now also J6.1 (Pin_1)
- new net SS: J6.4 (Pin_4), U3.12 (PB2)
Other:
- note removed: "Hall Count"
Changed lines of the file:
@@
 Sheet 1 1
 Title "microBoSL Board"
-Date "2021-04-23"
+Date "2021-05-03"
 Rev "0.2.0"
 Comp ""
@@
 	0    -1   -1   0
 $EndComp
-$Comp
-L power:GND #PWR05
-U 1 1 5D397783
-P 1750 4400
-F 0 "#PWR05" H 1750 4150 50  0001 C CNN
-F 1 "GND" V 1750 4225 50  0000 C CNN
-F 2 "" H 1750 4400 50  0000 C CNN
-F 3 "" H 1750 4400 50  0000 C CNN
-	1    1750 4400
-	0    1    1    0
-$EndComp
 Text GLabel 6800 5800 2    60   Input ~ 0
 D7
@@
 	0    1    1    0
 $EndComp
-$Comp
-L power:VPP #PWR07
-U 1 1 5D3B4E69
-P 1750 5000
-F 0 "#PWR07" H 1750 4850 50  0001 C CNN
-F 1 "VPP" V 1750 5200 50  0000 C CNN
-F 2 "" H 1750 5000 50  0000 C CNN
-F 3 "" H 1750 5000 50  0000 C CNN
-	1    1750 5000
-	0    -1   -1   0
-$EndComp
 Text GLabel 1750 5200 0    60   Input ~ 0
 V_3.3
@@
 Text GLabel 6800 5500 2    60   Input ~ 0
 D4
-Text GLabel 6800 3400 2    60   Input ~ 0
-D8
+Text GLabel 6800 3600 2    60   Input ~ 0
+SS
 Text GLabel 6800 3700 2    60   Input ~ 0
-D11
+MOSI
 Text GLabel 6800 3800 2    60   Input ~ 0
-D12
+MISO
 Text GLabel 6800 3900 2    60   Input ~ 0
-D13
+SCLK
 $Comp
 L Device:R R3
@@
 Text Notes 3400 3950 3    60   ~ 0
 Hall Wake
-Text Notes 3550 3950 3    60   ~ 0
-Hall Count
 Text GLabel 6800 5600 2    60   Input ~ 0
 Hall_WKE_P
@@
 F 0 "J1" H 2030 3942 50  0000 L CNN
 F 1 "Conn_01x04" H 2030 3851 50  0000 L CNN
-F 2 "Connector_PinHeader_2.54mm:PinHeader_1x04_P2.54mm_Vertical" H 1950 3950 50  0001 C CNN
+F 2 "Connector_PinHeader_1.27mm:PinHeader_1x04_P1.27mm_Vertical" H 1950 3950 50  0001 C CNN
 F 3 "~" H 1950 3950 50  0001 C CNN
 	1    1950 3950
@@
 $EndComp
 $Comp
-L Connector_Generic:Conn_01x04 J2
-U 1 1 5FD316A6
-P 1950 4500
-F 0 "J2" H 2030 4492 50  0000 L CNN
-F 1 "Conn_01x04" H 2030 4401 50  0000 L CNN
-F 2 "Connector_PinHeader_1.27mm:PinHeader_1x04_P1.27mm_Vertical" H 1950 4500 50  0001 C CNN
-F 3 "~" H 1950 4500 50  0001 C CNN
-	1    1950 4500
-	1    0    0    -1
-$EndComp
-Text GLabel 3300 4550 0    60   Input ~ 0
-D3
-Text GLabel 3300 4650 0    60   Input ~ 0
-D4
-Text GLabel 3300 4750 0    60   Input ~ 0
-D7
-Text GLabel 3300 4850 0    60   Input ~ 0
-D8
-Text GLabel 3300 4950 0    60   Input ~ 0
-D10
-Text GLabel 3300 5050 0    60   Input ~ 0
-D11
-Text GLabel 3300 5150 0    60   Input ~ 0
-D12
-Text GLabel 3300 5250 0    60   Input ~ 0
-D13
-$Comp
 L Connector_Generic:Conn_01x04 J3
 U 1 1 5FD35207
@@
 $EndComp
 $Comp
-L power:GND #PWR023
-U 1 1 5FDF7BF0
-P 8150 4200
-F 0 "#PWR023" H 8150 3950 50  0001 C CNN
-F 1 "GND" H 8150 4050 50  0000 C CNN
-F 2 "" H 8150 4200 50  0000 C CNN
-F 3 "" H 8150 4200 50  0000 C CNN
-	1    8150 4200
-	1    0    0    -1
-$EndComp
-$Comp
-L power:GND #PWR022
-U 1 1 5FDF7F7C
-P 8150 3800
-F 0 "#PWR022" H 8150 3550 50  0001 C CNN
-F 1 "GND" H 8150 3650 50  0000 C CNN
-F 2 "" H 8150 3800 50  0000 C CNN
-F 3 "" H 8150 3800 50  0000 C CNN
-	1    8150 3800
-	-1   0    0    1
-$EndComp
-$Comp
-L Device:Crystal_GND24 Y1
+L Device:Crystal Y1
 U 1 1 5FDFDAE8
 P 8150 4000
@@
 	-1   0    0    1
 $EndComp
-$Comp
-L Connector_Generic:Conn_01x10 J6
-U 1 1 5FE03C64
-P 3500 4950
-F 0 "J6" H 3580 4942 50  0000 L CNN
-F 1 "Conn_01x10" H 3580 4851 50  0000 L CNN
-F 2 "Connector_PinHeader_1.27mm:PinHeader_1x10_P1.27mm_Vertical" H 3500 4950 50  0001 C CNN
-F 3 "~" H 3500 4950 50  0001 C CNN
-	1    3500 4950
-	1    0    0    -1
-$EndComp
-Text GLabel 3300 5450 0    60   Input ~ 0
-A3
-Text GLabel 3300 5350 0    60   Input ~ 0
-A1
 $Comp
 L power:GND #PWR041
@@
 	1    0    0    -1
 $EndComp
-Text GLabel 6800 3600 2    60   Input ~ 0
+Text GLabel 6800 3400 2    60   Input ~ 0
 MREV
 Text GLabel 6100 1225 0    60   Input ~ 0
@@
 	8500 4000 8500 4100
 Wire Wire Line
-	7925 4100 7925 4450
-Wire Wire Line
-	7925 4450 8375 4450
-Wire Wire Line
-	8375 4450 8375 4100
+	7925 4100 7925 4200
+Wire Wire Line
+	7925 4200 8375 4200
+Wire Wire Line
+	8375 4200 8375 4100
 Wire Wire Line
 	8375 4100 8500 4100
@@
 Wire Wire Line
 	2650 1650 3175 1650
+$Comp
+L Connector_Generic:Conn_01x04 J6
+U 1 1 609936C2
+P 3500 4650
+F 0 "J6" H 3580 4642 50  0000 L CNN
+F 1 "Conn_01x04" H 3580 4551 50  0000 L CNN
+F 2 "Connector_PinHeader_1.27mm:PinHeader_1x04_P1.27mm_Vertical" H 3500 4650 50  0001 C CNN
+F 3 "~" H 3500 4650 50  0001 C CNN
+	1    3500 4650
+	1    0    0    -1
+$EndComp
+Text GLabel 3300 4850 0    60   Input ~ 0
+SS
+Text GLabel 3300 4750 0    60   Input ~ 0
+MOSI
+Text GLabel 3300 4650 0    60   Input ~ 0
+MISO
+Text GLabel 3300 4550 0    60   Input ~ 0
+SCLK
+$Comp
+L Connector_Generic:Conn_01x03 J2
+U 1 1 609EBDCD
+P 1950 4600
+F 0 "J2" H 2030 4642 50  0000 L CNN
+F 1 "Conn_01x03" H 2030 4551 50  0000 L CNN
+F 2 "Connector_PinHeader_1.27mm:PinHeader_1x03_P1.27mm_Vertical" H 1950 4600 50  0001 C CNN
+F 3 "~" H 1950 4600 50  0001 C CNN
+	1    1950 4600
+	1    0    0    -1
+$EndComp
+Text GLabel 1750 5000 0    60   Input ~ 0
+VBAT
 $EndSCHEMATC
