File: micro/EDA/EDA/microBoSL.sch (KiCad schematic (older format))
At the start: 54 parts, among them J1 Conn_01x04, J10 MOTOR_OUT, J11 Conn_01x03, J12 Conn_01x03, J13 Conn_01x03, J2 Conn_01x03, J3 Conn_01x04, J4 BATTERY CONN, J5 Conn_01x03, J6 Conn_01x04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

Commit message: fixed power switch on microBoSL added o-ring fix pinout
Parts:
- removed U1, U2: TPS709A33DBVT, Package_TO_SOT_SMD:SOT-23-5, symbol microBoSL-rescue:TPS709A33DBVT
- added U1, U2: MAX40203ANS, Package_BGA:WLP-4_0.73x0.73mm_Layout2x2_P0.35mm_Ball0.22mm_Pad0.2mm_NSMD, symbol Analog_Switch:MAX40200ANS
- added U10: TPS709A33DBVT, Package_TO_SOT_SMD:SOT-23-5, symbol microBoSL-rescue:TPS709A33DBVT
- Y1: footprint Crystal:Crystal_SMD_5032-2Pin_5.0x3.2mm -> Crystal:Crystal_SMD_5032-4Pin_5.0x3.2mm; symbol Device:Crystal -> Device:Crystal_GND24
Connections:
- net GND: now also J11.2 (Pin_2), J12.2 (Pin_2), J13.2 (Pin_2), J5.2 (Pin_2), Y1.2, Y1.4, U1.B2 (GND), U10.2 (GND), U2.B2 (GND); no longer J11.1 (Pin_1), J12.1 (Pin_1), J13.1 (Pin_1), J5.1 (Pin_1)
- net Hall_MA_S: now also J11.1 (Pin_1); no longer J11.2 (Pin_2)
- net Hall_MB_S: now also J12.3 (Pin_3); no longer J12.2 (Pin_2)
- net Hall_MC_S: now also J13.3 (Pin_3); no longer J13.2 (Pin_2)
- net Hall_P: no longer J12.3 (Pin_3), J13.3 (Pin_3)
- net Hall_WKE_S: now also J5.1 (Pin_1); no longer J5.2 (Pin_2)
- net TLL_RST: now also J6.4 (Pin_4)
- net USB_V: now also U1.A1 (VDD), U1.B1 (EN)
- net VBAT: now also Q1.3 (D), U2.A1 (VDD), U2.B1 (EN); no longer Q1.2 (S)
- net VPP: now also Q1.2 (S); no longer Q1.3 (D)
- net V_3.3: now also U10.1 (OUT)
- net at C5.2, U3.5 (XTAL1/PB6): now also Y1.3; no longer Y1.2
- net SS renamed Hall_P2
- net Hall_P2: now also J12.1 (Pin_1), J13.1 (Pin_1); no longer J6.4 (Pin_4)
- new net: U1.A2 (OUT), U10.3 (IN), U2.A2 (OUT)
- no-connect marks 19 -> 18
Other:
- note added: "Battery Switch"
- moved on the sheet: C1, C12, C13, C14, C2, C3, C4, C5, C6, C7, C8, C9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
