File: micro/EDA/EDA/microBoSL.kicad_pcb (KiCad board)
At the start: 4 copper layers, 45 x 15 mm, 60 parts, among them J1 Conn_01x04, J10 MOTOR_OUT, J11 Conn_01x03, J12 Conn_01x03, J13 Conn_01x03, J2 Conn_01x03, J3 Conn_01x04, J4 BATTERY CONN, J5 Conn_01x03, J6 Conn_01x04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

Commit message: fixed power switch on microBoSL added o-ring fix pinout
Parts:
- removed REF** (x6): Fiducial_1mm_Mask2mm, Fiducial:Fiducial_1mm_Mask2mm
- added U10: TPS709A33DBVT, Package_TO_SOT_SMD:SOT-23-5, B.Cu at (106.8, 112.6)
- U1, U2: value TPS709A33DBVT -> MAX40203ANS; footprint Package_TO_SOT_SMD:SOT-23-5 -> Package_BGA:WLP-4_0.73x0.73mm_Layout2x2_P0.35mm_Ball0.22mm_Pad0.2mm_NSMD
- Y1: footprint Crystal:Crystal_SMD_5032-2Pin_5.0x3.2mm -> Crystal:Crystal_SMD_5032-4Pin_5.0x3.2mm
- moved U1 2.86 mm to (106.4, 109.8), turned to 0 degrees
- moved U2 2.09 mm to (109.1, 109.8), turned to 270 degrees
- moved Q1 0.68 mm to (106.5, 107.5), turned to 0 degrees
- renumbered RST to SW1
Connections:
- J11 pad 1: GND -> Hall_MA_S
- J11 pad 2: Hall_MA_S -> GND
- J12 pad 1: GND -> Hall_P2
- J12 pad 2: Hall_MB_S -> GND
- J12 pad 3: Hall_P -> Hall_MB_S
- J13 pad 1: GND -> Hall_P2
- J13 pad 2: Hall_MC_S -> GND
- J13 pad 3: Hall_P -> Hall_MC_S
- J5 pad 1: GND -> Hall_WKE_S
- J5 pad 2: Hall_WKE_S -> GND
- J6 pad 4: SS -> TLL_RST
- Q1 pad 2: VBAT -> VPP
- Q1 pad 3: VPP -> VBAT
- U3 pad 12: SS -> Hall_P2
- Y1 pad 2: Net-(C5-Pad2) -> GND
Routing:
- net Hall_P2: track 0.00 -> 23.7 mm, vias 0 -> 1
- net Hall_P: track 43.5 -> 24.3 mm
- net SS: track 16.2 -> 0.00 mm, vias 1 -> 0
- net Net-(U1-PadA2): track 0.00 -> 6.75 mm
- net GND: track 117.3 -> 111.3 mm, vias 12 -> 14
- net Net-(Q1-Pad1): track 1.22 -> 4.38 mm
- net Hall_WKE_S: track 21.6 -> 24.0 mm
- net Hall_MA_S: track 15.8 -> 14.2 mm
- net TLL_RST: track 45.8 -> 47.3 mm
- net MOSI: track 15.4 -> 14.2 mm
- net USB_V: track 13.9 -> 14.9 mm
- net Net-(C6-Pad2): track 15.1 -> 16.0 mm
- net SCLK: track 17.8 -> 16.9 mm
- net Net-(C5-Pad2): track 5.36 -> 4.57 mm
- net SDA: track 20.1 -> 20.9 mm
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Other:
- board text added: "ON"
- board text removed: "SS"
